File: controller2/controller2.kicad_pcb (KiCad board)
At the start: 2 copper layers, 113.5 x 60.5 mm, 49 parts, among them J1 5V_IN, J2 Conn_02x17_Odd_Even, J3 VCC_IN, J4 Conn_01x10, Q1 Q_NMOS_GSD, U1 R-78E3.3-0.5, U2 TLP127, U3 ADM2482, U4 TLP127, U5 TLP127, U6 R-78E3.3-0.5

Commit message: No commit no cry. Controller IO isolation board is ready for manufacturing
Parts:
- added C10: C, Capacitors_SMD:C_0603_HandSoldering, B.Cu at (219.0, 69.8)
- added C13: C, Capacitors_SMD:C_0603_HandSoldering, B.Cu at (212.2, 73.2)
- added D10: D_Small, Diodes_SMD:D_SOD-323_HandSoldering, B.Cu at (164.0, 81.8)
- added D12: D_Small, Diodes_SMD:D_SOD-323_HandSoldering, B.Cu at (175.5, 70.0)
- added D13: SMCJ12CA, Diodes_SMD:DO-214AB_Handsoldering, B.Cu at (216.0, 66.5)
- added D14: SMCJ12CA, Diodes_SMD:DO-214AB_Handsoldering, B.Cu at (209.2, 68.2)
- added D3: D_Small, Diodes_SMD:D_SOD-323_HandSoldering, B.Cu at (164.0, 76.0)
- added Q2: Q_NMOS_GSD, TO_SOT_Packages_THT:TO-220-3_Vertical, F.Cu at (219.5, 83.3)
- added R16: R, Resistors_SMD:R_0603_HandSoldering, B.Cu at (162.0, 76.0)
- added R17: R, Resistors_SMD:R_0603_HandSoldering, B.Cu at (152.2, 87.2)
- added R18: R, Resistors_SMD:R_0603_HandSoldering, B.Cu at (178.5, 71.5)
- added R19: R, Resistors_SMD:R_0603_HandSoldering, B.Cu at (221.5, 80.8)
- added R20: R_Small, Resistors_SMD:R_0603_HandSoldering, B.Cu at (221.5, 76.5)
- added R21: R_Small, Resistors_SMD:R_0603_HandSoldering, B.Cu at (221.5, 70.8)
- added U7: TLP222A, Housings_DIP:DIP-4_W7.62mm, F.Cu at (165.9, 74.5)
- added U8: TLP222A, Housings_DIP:DIP-4_W7.62mm, F.Cu at (173.5, 71.0)
- J3: value VCC_IN -> Conn_01x06; footprint door:TerminalBlock_WAGO-205_2pol -> door:TerminalBlock_WAGO-205_10pol
- U2, U4, U5: value TLP127 -> TLP222A; footprint Housings_SSOP:MFSOP6-4_4.4x3.6mm_Pitch1.27mm -> Housings_DIP:DIP-4_W7.62mm; moved to F.Cu
- moved C1 46.3 mm to (163.8, 118.5), turned to 90 degrees
- moved C4 19.6 mm to (203.0, 60.0)
- moved R3 17.9 mm to (147.8, 81.0), turned to 270 degrees
- moved R4 15.3 mm to (161.0, 110.0), turned to 90 degrees
- moved D8 13.5 mm to (178.0, 61.0)
- moved C9 12.0 mm to (182.0, 68.0)
- moved F1 10.8 mm to (231.5, 58.5)
- moved J3 9.30 mm to (231.0, 65.0)
- moved C11 8.00 mm to (199.5, 72.0)
- moved C12 8.00 mm to (190.5, 72.0)
- moved D11 8.00 mm to (186.0, 66.5)
- moved D9 8.00 mm to (195.0, 66.5)
- moved U2 6.45 mm to (165.9, 80.5), turned to 0 degrees
- moved U4 3.16 mm to (173.5, 95.0)
- moved U5 3.04 mm to (173.5, 89.0)
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Connections:
- J2 pad 12: Net-(J2-Pad12) -> /AUX_IN_ISO
- J2 pad 13: Net-(J2-Pad13) -> /AUX_OUT_ISO
- R1 pad 1: Net-(R1-Pad1) -> Net-(D10-Pad1)
- U2 pad 1: VCC -> Net-(D10-Pad1)
- U2 pad 4: GND -> VCC
- U4 pad 3: GNDD -> GND
- U4 pad 4: GND -> /~SWITCH_ISO
- U5 pad 3: GNDD -> GND
- U5 pad 4: GND -> /~VCC_GOOD
Routing:
- net /AUX_IN: track 0.00 -> 65.6 mm
- net VCC: track 156.8 -> 213.4 mm, vias 6 -> 8
- net Net-(Q2-Pad1): track 0.00 -> 54.7 mm
- net /AUX_IN_ISO: track 0.00 -> 39.5 mm, vias 0 -> 2
- net GNDD: track 0.00 -> 32.1 mm, vias 0 -> 2
- net /AUX_OUT_ISO: track 0.00 -> 30.8 mm, vias 0 -> 2
- net GND: track 2.08 -> 31.0 mm, vias 0 -> 4
- net /AUX_OUT: track 0.00 -> 18.6 mm, vias 0 -> 2
- net /BUZZ_LED: track 49.6 -> 67.0 mm, vias 0 -> 2
- net /SWITCH: track 60.9 -> 76.3 mm
- net Net-(J3-Pad3): track 0.00 -> 8.59 mm
- net Net-(J3-Pad5): track 0.00 -> 8.52 mm
- net Net-(J4-Pad9): track 0.00 -> 8.40 mm
- net Net-(J4-Pad7): track 0.00 -> 8.40 mm
- net Net-(J4-Pad5): track 0.00 -> 8.40 mm
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Other:
- board size 113.5 x 60.5 mm -> 113.5 x 70.5 mm
- board text added: "TECHNARIUM 2017"
