File: controller2/controller2.sch (KiCad schematic (older format))
At the start: 49 parts, among them J1 5V_IN, J2 Conn_02x17_Odd_Even, J3 VCC_IN, J4 Conn_01x10, Q1 Q_NMOS_GSD, U1 R-78E3.3-0.5, U2 TLP127, U3 ADM2482, U4 TLP127, U5 TLP127, U6 R-78E3.3-0.5

Commit message: No commit no cry. Controller IO isolation board is ready for manufacturing
Parts:
- removed J3: VCC_IN, door:TerminalBlock_WAGO-205_2pol, symbol Connector:Conn_01x02
- removed U2, U4, U5: TLP127, Housings_SSOP:MFSOP6-4_4.4x3.6mm_Pitch1.27mm, symbol opto:TLP127
- added C10, C13: C, Capacitors_SMD:C_0603_HandSoldering, symbol device:C
- added D10, D12, D3: D_Small, Diodes_SMD:D_SOD-323_HandSoldering, symbol device:D_Small
- added D13, D14: SMCJ12CA, Diodes_SMD:DO-214AB_Handsoldering, symbol device:D_TVS
- added J3: Conn_01x06, door:TerminalBlock_WAGO-205_10pol, symbol Connector:Conn_01x06
- added Q2: Q_NMOS_GSD, TO_SOT_Packages_THT:TO-220-3_Vertical, symbol device:Q_NMOS_GDS
- added R16, R17, R18, R19: R, Resistors_SMD:R_0603_HandSoldering, symbol device:R
- added R20, R21: R_Small, Resistors_SMD:R_0603_HandSoldering, symbol device:R_Small
- added U2, U4, U5, U7, U8: TLP222A, Housings_DIP:DIP-4_W7.62mm, symbol opto:TLP222A
Connections:
- net labels added: AUX_IN, AUX_IN_ISO, AUX_OUT, AUX_OUT_ISO
- wire segments 122 -> 157
Other:
- moved on the sheet: C1, D2, F1, J1, J2, MK1, MK2, R2, R3, R4, R6, U1
